File: WFH_BOARD.kicad_pcb (KiCad board)
At the start: 2 copper layers, 95.7 x 98.3 mm, 55 parts, among them J1 USB_B, J2 Conn_01x06_Male, J3 Conn_01x05_Male, J4 Conn_01x01, J5 Conn_01x03_Female, J6 Conn_01x03_Female, J7 Conn_01x03_Female, J8 Conn_01x01, J9 Conn_01x01, K1 G5LE-1, K2 G5LE-1, K3 G5LE-1, Q1 BC547, Q2 BC547, Q3 BC547, U1 4N25, U2 4N25, U3 4N25, U4 FT232RL, U5 ATmega328-AU, Y1 Crystal

Commit message: Final modifications
Other:
- board text added: "WFH board V1.0 version"
- board text removed: "WFH board COVID edition"
Changed lines of the file:
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@@
   (general
     (thickness 1.6)
-    (drawings 17)
+    (drawings 13)
     (tracks 467)
     (zones 0)
@@
     (32 B.Adhes user)
     (33 F.Adhes user)
-    (34 B.Paste user hide)
+    (34 B.Paste user)
     (35 F.Paste user)
     (36 B.SilkS user)
-    (37 F.SilkS user hide)
+    (37 F.SilkS user)
     (38 B.Mask user)
     (39 F.Mask user)
@@
   (gr_line (start 102 137) (end 135 137) (layer Edge.Cuts) (width 0.1))
   (gr_line (start 102 136) (end 102 137) (layer Edge.Cuts) (width 0.1))
-  (gr_arc (start 94.615 158.115) (end 95.249999 160.654999) (angle -147.5288077) (layer F.SilkS) (width 0.12))
-  (gr_arc (start 97.155 156.845) (end 95.250001 158.114999) (angle -146.3099325) (layer F.SilkS) (width 0.12))
-  (gr_circle (center 91.44 155.575) (end 104.775 160.02) (layer F.SilkS) (width 0.12))
-  (gr_circle (center 93.45 138.5) (end 94.1 140.95) (layer F.SilkS) (width 0.12))
   (gr_text 2020 (at 71.7 116.2) (layer F.Cu)
     (effects (font (size 1.1 1.1) (thickness 0.275)))
@@
     (effects (font (size 1.1 1.1) (thickness 0.275)))
   )
-  (gr_text "WFH board\n COVID edition" (at 119.1 48.5) (layer F.Cu)
+  (gr_text "WFH board\n V1.0 version" (at 119.1 48.5) (layer F.Cu)
     (effects (font (size 1.5 1.5) (thickness 0.3)))
   )
